File: arc40.kicad_pcb (KiCad board)
At the start: 2 copper layers, 85 parts, among them U1 ProMicro

Commit message: added a small little detail called board edges
Other:
- board outline added: 238.1 x 76.2 mm
